File: AD5791-AD7734/arduino-shield/arduino-shield.sch (EAGLE design)
At the start: 27 parts, among them IC1 74ABT125PW, IC2 74ABT125PW, X1 22-23-2021, X2 22-23-2021, X3 22-23-2021, X4 22-23-2021, X5 22-23-2021

Commit message: Part numbers renumbered.
Parts:
- C1: value 1uF -> 0.1uF
- C2: value 1.5uF -> 0.1uF
- C3: value 0.1uF -> 1uF
- C4: value 0.1uF -> 1.5uF
- R1, R2: value 300 mR -> 330 mR
- renumbered ADC0 to SV5, DAC0 to SV1, DAC1 to SV2, DAC2 to SV3, DAC3 to SV4
Connections:
- net AGND: now also C3.2, C4.2, X4-2.S, X5-2.S; no longer C1.2, C2.2, X1-2.S, X2-2.S
- net GND: now also C1.2, C2.2, X1-2.S, X2-2.S; no longer C3.2, C4.2, X4-2.S, X5-2.S
- net N$1: now also C3.1, X4-1.S; no longer C1.1, X1-1.S
- net N$2: now also C4.1, X5-1.S; no longer C2.1, X2-1.S
- net N$4: now also X2-1.S; no longer X3-1.S
- net N$7: now also X3-1.S; no longer X4-1.S
- net VCC: now also C1.1, C2.1, X1-1.S; no longer C3.1, C4.1, X5-1.S
